File: schematics/Uzebox-Omega/V1.1.1/Uzebox Game Console Omega.brd (EAGLE design)
At the start: 100 x 81 mm, 91 parts, among them CON1 USBSERIALSMD, IC1 MCP1700, IC2 7805T, U5 DC IN, U6 23LC1024, X1 A/V

Commit message: Update schematic
Parts:
- renumbered MCU to ATMEGA644A-PU, X1 to KMDGX-9S-N
